File: PCB/MacropadV1.kicad_pcb (KiCad board)
At the start: 2 copper layers, 59 x 59 mm, 17 parts, among them J1 Conn_01x04, SW1 SW_Push, SW10 RotaryEncoder_Switch, SW2 SW_Push, SW3 SW_Push, SW4 SW_Push, SW5 SW_Push, SW6 SW_Push, U1 MOUDLE-SEEEDUINO-XIAO

Commit message: just making sure i didnt forget anything
Parts:
- D1, D2, D3, D4, D5, D6: value D -> 1N4148; footprint Crystal:Crystal_SMD_G8-2Pin_3.2x1.5mm -> Diode_SMD:D_SOD-123
- moved D5 5.55 mm to (57.3, 38.5)
Routing:
- net row2: track 26.8 -> 31.5 mm
- net Net-(D5-A): track 3.52 -> 7.29 mm
- net Net-(D6-A): track 11.1 -> 10.1 mm
- net row1: track 25.1 -> 24.4 mm

Commit message: added a silkscreen image and added gerber files
Parts:
- added G***: LOGO, KicadMods:HobbesPCBLogo, B.Cu at (67.2, 59.5)
