File: PCB/MacropadV1.kicad_pcb (KiCad board)
At the start: 2 copper layers, 59 x 59 mm, 18 parts, among them J1 Conn_01x04, SW1 SW_Push, SW10 RotaryEncoder_Switch, SW2 SW_Push, SW3 SW_Push, SW4 SW_Push, SW5 SW_Push, SW6 SW_Push, U1 MOUDLE-SEEEDUINO-XIAO

Commit message: fixed schematic display error
Connections:
- J1 pad 1: Net-(J1-Pin_1) -> GND
- J1 pad 2: Net-(J1-Pin_2) -> VCC
- J1 pad 3: GND -> Net-(J1-Pin_3)
- J1 pad 4: VCC -> Net-(J1-Pin_4)
- R1 pad 1: Net-(J1-Pin_2) -> Net-(J1-Pin_4)
- R2 pad 1: Net-(J1-Pin_1) -> Net-(J1-Pin_3)
Routing:
- net Net-(J1-Pin_3): track 0.00 -> 14.1 mm
- net Net-(J1-Pin_2): track 8.07 -> 0.00 mm
- net Net-(J1-Pin_1): track 7.78 -> 0.00 mm
- net GND: track 78.4 -> 83.4 mm
- net Net-(J1-Pin_4): track 0.00 -> 4.33 mm
- net VCC: track 140.5 -> 142.6 mm
Changed lines of the file:
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@@
 			(layers "*.Cu" "*.Mask")
 			(remove_unused_layers no)
-			(net "Net-(J1-Pin_1)")
+			(net "GND")
 			(pinfunction "Pin_1_1")
 			(pintype "passive")
@@
 			(layers "*.Cu" "*.Mask")
 			(remove_unused_layers no)
-			(net "Net-(J1-Pin_2)")
+			(net "VCC")
 			(pinfunction "Pin_2_2")
 			(pintype "passive")
@@
 			(layers "*.Cu" "*.Mask")
 			(remove_unused_layers no)
-			(net "GND")
+			(net "Net-(J1-Pin_3)")
 			(pinfunction "Pin_3_3")
 			(pintype "passive")
@@
 			(layers "*.Cu" "*.Mask")
 			(remove_unused_layers no)
-			(net "VCC")
+			(net "Net-(J1-Pin_4)")
 			(pinfunction "Pin_4_4")
 			(pintype "passive")
@@
 			(layers "*.Cu" "*.Mask")
 			(remove_unused_layers no)
-			(net "Net-(J1-Pin_2)")
+			(net "Net-(J1-Pin_4)")
 			(pintype "passive")
 		)
@@
 			(layers "*.Cu" "*.Mask")
 			(remove_unused_layers no)
-			(net "Net-(J1-Pin_1)")
+			(net "Net-(J1-Pin_3)")
 			(pintype "passive")
 		)
@@
 	)
 	(segment
+		(start 67.605 38.15)
+		(end 74.435635 38.15)
+		(width 0.2)
+		(layer "F.Cu")
+		(net "GND")
+	)
+	(segment
+		(start 76.25 36.335635)
+		(end 76.25 30.7)
+		(width 0.2)
+		(layer "F.Cu")
+		(net "GND")
+	)
+	(segment
+		(start 65.305 40.45)
+		(end 67.605 38.15)
+		(width 0.2)
+		(layer "F.Cu")
+		(net "GND")
+	)
+	(segment
+		(start 72.75 27.2)
+		(end 60.75 27.2)
+		(width 0.2)
+		(layer "F.Cu")
+		(net "GND")
+	)
+	(segment
+		(start 58.7 20.05)
+		(end 27.64 20.05)
+		(width 0.2)
+		(layer "F.Cu")
+		(net "GND")
+	)
+	(segment
+		(start 74.435635 38.15)
+		(end 76.25 36.335635)
+		(width 0.2)
+		(layer "F.Cu")
+		(net "GND")
+	)
+	(segment
+		(start 75.25 29.7)
+		(end 72.75 27.2)
+		(width 0.2)
+		(layer "F.Cu")
+		(net "GND")
+	)
+	(segment
+		(start 27.64 20.05)
+		(end 21.95 25.74)
+		(width 0.2)
+		(layer "F.Cu")
+		(net "GND")
+	)
+	(segment
+		(start 76.25 30.7)
+		(end 75.25 29.7)
+		(width 0.2)
+		(layer "F.Cu")
+		(net "GND")
+	)
+	(segment
+		(start 62.05 23.4)
+		(end 58.7 20.05)
+		(width 0.2)
+		(layer "F.Cu")
+		(net "GND")
+	)
+	(segment
+		(start 62.05 25.9)
+		(end 62.05 23.4)
+		(width 0.2)
+		(layer "F.Cu")
+		(net "GND")
+	)
+	(segment
+		(start 60.75 27.2)
+		(end 62.05 25.9)
+		(width 0.2)
+		(layer "F.Cu")
+		(net "GND")
+	)
+	(segment
+		(start 72.89 77.11)
+		(end 72.75 77.25)
+		(width 0.2)
+		(layer "F.Cu")
+		(net "VCC")
+	)
+	(segment
+		(start 27.25 31.048529)
+		(end 27.25 30.551471)
+		(width 0.2)
+		(layer "F.Cu")
+		(net "VCC")
+	)
+	(segment
+		(start 24.978529 28.28)
+		(end 21.95 28.28)
+		(width 0.2)
+		(layer "F.Cu")
+		(net "VCC")
+	)
+	(segment
+		(start 27.25 30.551471)
+		(end 24.978529 28.28)
+		(width 0.2)
+		(layer "F.Cu")
+		(net "VCC")
+	)
+	(segment
+		(start 72.75 77.25)
+		(end 24.25 77.25)
+		(width 0.2)
+		(layer "F.Cu")
+		(net "VCC")
+	)
+	(segment
+		(start 23.07 35.228529)
+		(end 27.25 31.048529)
+		(width 0.2)
+		(layer "F.Cu")
+		(net "VCC")
+	)
+	(segment
+		(start 23.07 76.07)
+		(end 23.07 35.228529)
+		(width 0.2)
+		(layer "F.Cu")
+		(net "VCC")
+	)
+	(segment
+		(start 72.89 45.494999)
+		(end 72.89 77.11)
+		(width 0.2)
+		(layer "F.Cu")
+		(net "VCC")
+	)
+	(segment
+		(start 24.25 77.25)
+		(end 23.07 76.07)
+		(width 0.2)
+		(layer "F.Cu")
+		(net "VCC")
+	)
+	(segment
+		(start 67.845001 40.45)
+		(end 72.89 45.494999)
+		(width 0.2)
+		(layer "F.Cu")
+		(net "VCC")
+	)
+	(segment
 		(start 45.22 32.97)
 		(end 45.22 27.07)
@@
 	)
 	(segment
-		(start 71.560001 36.7)
-		(end 74.33 36.7)
-		(width 0.2)
-		(layer "F.Cu")
-		(net "Net-(J1-Pin_2)")
-	)
-	(segment
-		(start 67.810001 40.45)
-		(end 71.560001 36.7)
-		(width 0.2)
-		(layer "F.Cu")
-		(net "Net-(J1-Pin_2)")
-	)
-	(segment
 		(start 45.00353 71.032)
 		(end 36.05 62.07847)
@@
 	)
 	(segment
-		(start 65.27 40.45)
-		(end 65.27 41.91)
-		(width 0.2)
-		(layer "F.Cu")
-		(net "Net-(J1-Pin_1)")
-	)
-	(segment
-		(start 65.27 41.91)
-		(end 60.8 46.38)
-		(width 0.2)
-		(layer "F.Cu")
-		(net "Net-(J1-Pin_1)")
-	)
-	(segment
-		(start 76.25 36.335635)
-		(end 76.25 30.7)
-		(width 0.2)
-		(layer "F.Cu")
-		(net "GND")
-	)
-	(segment
-		(start 72.75 27.2)
-		(end 60.75 27.2)
-		(width 0.2)
-		(layer "F.Cu")
-		(net "GND")
-	)
-	(segment
-		(start 58.7 20.05)
-		(end 27.64 20.05)
-		(width 0.2)
-		(layer "F.Cu")
-		(net "GND")
-	)
-	(segment
-		(start 70.35 40.45)
-		(end 73 37.8)
-		(width 0.2)
-		(layer "F.Cu")
-		(net "GND")
-	)
-	(segment
-		(start 75.25 29.7)
-		(end 72.75 27.2)
-		(width 0.2)
-		(layer "F.Cu")
-		(net "GND")
-	)
-	(segment
-		(start 27.64 20.05)
-		(end 21.95 25.74)
-		(width 0.2)
-		(layer "F.Cu")
-		(net "GND")
-	)
-	(segment
-		(start 73 37.8)
-		(end 74.785635 37.8)
-		(width 0.2)
-		(layer "F.Cu")
-		(net "GND")
-	)
-	(segment
-		(start 76.25 30.7)
-		(end 75.25 29.7)
-		(width 0.2)
-		(layer "F.Cu")
-		(net "GND")
-	)
-	(segment
-		(start 74.785635 37.8)
-		(end 76.25 36.335635)
-		(width 0.2)
-		(layer "F.Cu")
-		(net "GND")
-	)
-	(segment
-		(start 62.05 23.4)
-		(end 58.7 20.05)
-		(width 0.2)
-		(layer "F.Cu")
-		(net "GND")
-	)
-	(segment
-		(start 62.05 25.9)
-		(end 62.05 23.4)
-		(width 0.2)
-		(layer "F.Cu")
-		(net "GND")
-	)
-	(segment
-		(start 60.75 27.2)
-		(end 62.05 25.9)
-		(width 0.2)
-		(layer "F.Cu")
-		(net "GND")
-	)
-	(segment
-		(start 72.89 77.11)
-		(end 72.75 77.25)
-		(width 0.2)
-		(layer "F.Cu")
-		(net "VCC")
-	)
-	(segment
-		(start 27.25 31.048529)
-		(end 27.25 30.551471)
-		(width 0.2)
-		(layer "F.Cu")
-		(net "VCC")
-	)
-	(segment
-		(start 24.978529 28.28)
-		(end 21.95 28.28)
-		(width 0.2)
-		(layer "F.Cu")
-		(net "VCC")
-	)
-	(segment
-		(start 72.89 40.45)
-		(end 72.89 77.11)
-		(width 0.2)
-		(layer "F.Cu")
-		(net "VCC")
-	)
-	(segment
-		(start 27.25 30.551471)
-		(end 24.978529 28.28)
-		(width 0.2)
-		(layer "F.Cu")
-		(net "VCC")
-	)
-	(segment
-		(start 72.75 77.25)
-		(end 24.25 77.25)
-		(width 0.2)
-		(layer "F.Cu")
-		(net "VCC")
-	)
-	(segment
-		(start 23.07 35.228529)
-		(end 27.25 31.048529)
-		(width 0.2)
-		(layer "F.Cu")
-		(net "VCC")
-	)
-	(segment
-		(start 23.07 76.07)
-		(end 23.07 35.228529)
-		(width 0.2)
-		(layer "F.Cu")
-		(net "VCC")
-	)
-	(segment
-		(start 24.25 77.25)
-		(end 23.07 76.07)
-		(width 0.2)
-		(layer "F.Cu")
-		(net "VCC")
-	)
-	(segment
 		(start 37.65 59.8)
 		(end 34.25 63.2)
@@
 		(net "Net-(U1-PB08_A6_D6_TX)")
 	)
+	(segment
+		(start 69.235 39.3)
+		(end 67.128654 39.3)
+		(width 0.2)
+		(layer "F.Cu")
+		(net "Net-(J1-Pin_3)")
+	)
+	(segment
+		(start 67.128654 39.3)
+		(end 66.455 39.973654)
+		(width 0.2)
+		(layer "F.Cu")
+		(net "Net-(J1-Pin_3)")
+	)
+	(segment
+		(start 66.455 41.85637)
+		(end 61.93137 46.38)
+		(width 0.2)
+		(layer "F.Cu")
+		(net "Net-(J1-Pin_3)")
+	)
+	(segment
+		(start 61.93137 46.38)
+		(end 60.8 46.38)
+		(width 0.2)
+		(layer "F.Cu")
+		(net "Net-(J1-Pin_3)")
+	)
+	(segment
+		(start 70.385 40.45)
+		(end 69.235 39.3)
+		(width 0.2)
+		(layer "F.Cu")
+		(net "Net-(J1-Pin_3)")
+	)
+	(segment
+		(start 66.455 39.973654)
+		(end 66.455 41.85637)
+		(width 0.2)
+		(layer "F.Cu")
+		(net "Net-(J1-Pin_3)")
+	)
+	(segment
+		(start 72.925 40.45)
+		(end 74.33 39.045)
+		(width 0.2)
+		(layer "B.Cu")
+		(net "Net-(J1-Pin_4)")
+	)
+	(segment
+		(start 74.33 39.045)
+		(end 74.33 36.7)
+		(width 0.2)
+		(layer "B.Cu")
+		(net "Net-(J1-Pin_4)")
+	)
 	(embedded_fonts no)

Commit message: added bom file
Connections:
- R1 pad 2: Net-(U1-PA9_A5_D5_SCL) -> Net-(U1-PA8_A4_D4_SDA)
- R2 pad 2: Net-(U1-PB08_A6_D6_TX) -> Net-(U1-PA9_A5_D5_SCL)
- U1 pad 10: col2 -> row2
- U1 pad 11: col1 -> row3
- U1 pad 3: row1 -> col1
- U1 pad 4: row2 -> col2
- U1 pad 5: row3 -> Net-(U1-PA8_A4_D4_SDA)
- U1 pad 7: Net-(U1-PB08_A6_D6_TX) -> unconnected-(U1-PB08_A6_D6_TX-Pad7)
- U1 pad 9: unconnected-(U1-PA7_A8_D8_SCK-Pad9) -> row1
Routing:
- net Net-(U1-PA8_A4_D4_SDA): track 0.00 -> 91.9 mm
- net Net-(U1-PA9_A5_D5_SCL): track 88.2 -> 25.8 mm, vias 0 -> 1
- net Net-(U1-PB08_A6_D6_TX): track 24.8 -> 0.00 mm, vias 2 -> 0
- net col1: track 65.0 -> 47.2 mm, vias 2 -> 0
- net row1: track 24.4 -> 38.9 mm, vias 0 -> 1
- net row2: track 31.5 -> 42.5 mm, vias 0 -> 3
- net row3: track 52.4 -> 44.3 mm, vias 0 -> 1
- net col2: track 53.4 -> 51.6 mm
